Commit message: working config

File: ROS2/src/controller/description/urdf/LBR3R760iisy.urdf (robot description, URDF)
Before this commit: robot LBR3R760iisy, 17 links, 16 joints
Joints:
- joint finger_joint: limit lower=-0.876 upper=0.876 effort=1000 velocity=2.0 -> lower=-0.876 upper=0.876 effort=1000 velocity=0.2
- joint left_inner_finger_joint: limit lower=-0.8757 upper=0.8757 effort=1000 velocity=2.0 -> lower=-0.8757 upper=0.8757 effort=1000 velocity=0.2
- joint left_inner_knuckle_joint: limit lower=-0.8757 upper=0.8757 effort=1000 velocity=2.0 -> lower=-0.8757 upper=0.8757 effort=1000 velocity=0.2
- joint right_inner_finger_joint: limit lower=-0.8757 upper=0.8757 effort=1000 velocity=2.0 -> lower=-0.8757 upper=0.8757 effort=1000 velocity=0.2
- joint right_inner_knuckle_joint: limit lower=-0.8757 upper=0.8757 effort=1000 velocity=2.0 -> lower=-0.8757 upper=0.8757 effort=1000 velocity=0.2
- joint right_outer_knuckle_joint: limit lower=-0.8757 upper=0.8757 effort=1000 velocity=2.0 -> lower=-0.8757 upper=0.8757 effort=1000 velocity=0.2

File: Webots/resource/LBR3R760iisy/LBR3R760iisy.urdf (robot description, URDF)
Before this commit: robot LBR3R760iisy, 17 links, 16 joints
Joints:
- joint finger_joint: limit lower=-0.876 upper=0.876 effort=1000 velocity=2.0 -> lower=-0.876 upper=0.876 effort=1000 velocity=0.2
- joint left_inner_finger_joint: limit lower=-0.8757 upper=0.8757 effort=1000 velocity=2.0 -> lower=-0.8757 upper=0.8757 effort=1000 velocity=0.2
- joint left_inner_knuckle_joint: limit lower=-0.8757 upper=0.8757 effort=1000 velocity=2.0 -> lower=-0.8757 upper=0.8757 effort=1000 velocity=0.2
- joint right_inner_finger_joint: limit lower=-0.8757 upper=0.8757 effort=1000 velocity=2.0 -> lower=-0.8757 upper=0.8757 effort=1000 velocity=0.2
- joint right_inner_knuckle_joint: limit lower=-0.8757 upper=0.8757 effort=1000 velocity=2.0 -> lower=-0.8757 upper=0.8757 effort=1000 velocity=0.2
- joint right_outer_knuckle_joint: limit lower=-0.8757 upper=0.8757 effort=1000 velocity=2.0 -> lower=-0.8757 upper=0.8757 effort=1000 velocity=0.2
